Commit message: ros2 control added

File: ur5_description/urdf/ur5.ros2_control.xacro (robot description, xacro)
@@ -1,148 +1,226 @@
 <?xml version="1.0"?>
 <robot xmlns:xacro="http://www.ros.org/wiki/xacro">
-  <xacro:macro name="ur5_ros2_control" params="prefix robot_ip local_ip use_fake_hardware:=^|false fake_sensor_commands:=^|false ">
-  <!-- initial_positions_file -->
-    <!-- <xacro:property name="initial_positions" value="${xacro.load_yaml(initial_positions_file)['initial_positions']}"/> -->
-    <ros2_control name="UR5HardwareInterface" type="system">
+  <xacro:macro name="ur5_ros2_control">
+    <gazebo>
+      <plugin name="gazebo_ros2_control" filename="libgazebo_ros2_control.so" >
+        <robot_param>robot_description</robot_param>
+        <robot_param_node>robot_state_publisher</robot_param_node>
+        <parameters>$(find gazebo_robot_sim)/config/robot_controllers.yaml</parameters>
+      </plugin>
+      <plugin name="gazebo_ros_ft_sensor_1" filename="libgazebo_ros_ft_sensor.so" >
+        <ros>
+          <namespace>/gazebo_sensors</namespace>
+          <remapping>wrench:=ft_sensor_1</remapping>
+        </ros>
+        <joint_name>joint1</joint_name>
+        <update_rate>50</update_rate>
+        <gaussian_noise>0.01</gaussian_noise>
+      </plugin>
+      <plugin name="gazebo_ros_ft_sensor_2" filename="libgazebo_ros_ft_sensor.so" >
+        <ros>
+          <namespace>/gazebo_sensors</namespace>
+          <remapping>wrench:=ft_sensor_2</remapping>
+        </ros>
+        <joint_name>joint2</joint_name>
+        <update_rate>50</update_rate>
+        <gaussian_noise>0.01</gaussian_noise>
+      </plugin>
+      <plugin name="gazebo_ros_ft_sensor_3" filename="libgazebo_ros_ft_sensor.so" >
+        <ros>
+          <namespace>/gazebo_sensors</namespace>
+          <remapping>wrench:=ft_sensor_3</remapping>
+        </ros>
+        <joint_name>joint3</joint_name>
+        <update_rate>50</update_rate>
+        <gaussian_noise>0.01</gaussian_noise>
+      </plugin>
+      <plugin name="gazebo_ros_ft_sensor_4" filename="libgazebo_ros_ft_sensor.so" >
+        <ros>
+          <namespace>/gazebo_sensors</namespace>
+          <remapping>wrench:=ft_sensor_4</remapping>
+        </ros>
+        <joint_name>joint4</joint_name>
+        <update_rate>50</update_rate>
+        <gaussian_noise>0.01</gaussian_noise>
+      </plugin>
+      <plugin name="gazebo_ros_ft_sensor_5" filename="libgazebo_ros_ft_sensor.so" >
+        <ros>
+          <namespace>/gazebo_sensors</namespace>
+          <remapping>wrench:=ft_sensor_5</remapping>
+        </ros>
+        <joint_name>joint5</joint_name>
+        <update_rate>50</update_rate>
+        <gaussian_noise>0.01</gaussian_noise>
+      </plugin>
+      <plugin name="gazebo_ros_ft_sensor_6" filename="libgazebo_ros_ft_sensor.so" >
+        <ros>
+          <namespace>/gazebo_sensors</namespace>
+          <remapping>wrench:=ft_sensor_6</remapping>
+        </ros>
+        <joint_name>joint6</joint_name>
+        <update_rate>50</update_rate>
+        <gaussian_noise>0.01</gaussian_noise>
+      </plugin>
+    </gazebo>
+    <gazebo reference="joint1">
+      <provideFeedback>true</provideFeedback>
+    </gazebo>
+    <gazebo reference="joint2">
+      <provideFeedback>true</provideFeedback>
+    </gazebo>
+    <gazebo reference="joint3">
+      <provideFeedback>true</provideFeedback>
+    </gazebo>
+    <gazebo reference="joint4">
+      <provideFeedback>true</provideFeedback>
+    </gazebo>
+    <gazebo reference="joint5">
+      <provideFeedback>true</provideFeedback>
+    </gazebo>
+    <gazebo reference="joint6">
+      <provideFeedback>true</provideFeedback>
+    </gazebo>
+    <ros2_control name="UR5_Arm_Hardware_Interface" type="system">
       <hardware>
-        <xacro:if value="${use_fake_hardware}">
-          <plugin>fake_components/GenericSystem</plugin>
-          <param name="fake_sensor_commands">${fake_sensor_commands}</param>
-          <param name="state_following_offset">0.0</param>
-        </xacro:if>
-        <xacro:unless value="${use_fake_hardware}">
-          <plugin>ur5_hardware/UR5HardwareInterface</plugin>
-          <param name="robot_ip">${robot_ip}</param>
-          <param name="local_ip">${local_ip}</param>
-        </xacro:unless>
+          <plugin>gazebo_ros2_control/GazeboSystem</plugin>
       </hardware>
-      <joint name="${prefix}joint1">
-        <command_interface name="position">
-          <param name="min">-2.7925</param>
-          <param name="max">2.7925</param>
-        </command_interface>
-        <command_interface name="velocity">
-          <param name="min">-4.0944</param>
-          <param name="max">4.0944</param>
-        </command_interface>
-        <command_interface name="effort"/>
-        <state_interface name="position"/>
-        <state_interface name="velocity"/>
-        <state_interface name="effort"/>
-        <!-- initial position for the FakeSystem -->
-        <!-- <param name="initial_position">${initial_positions['joint1']}</param>  -->
-        <param name="initial_position">0.0</param>
-      </joint>
-      <joint name="${prefix}joint2">
-        <command_interface name="position">
-          <param name="min">-2.7925</param>
-          <param name="max">2.7925</param>
-        </command_interface>
-        <command_interface name="velocity">
-          <param name="min">-4.0944</param>
-          <param name="max">4.0944</param>
-        </command_interface>
-        <command_interface name="effort"/>
-        <state_interface name="position"/>
-        <state_interface name="velocity"/>
-        <state_interface name="effort"/>
-        <!-- initial position for the FakeSystem -->
-        <param name="initial_position">0.0</param>
-        <!-- <param name="initial_position">${initial_positions['joint2']}</param>        -->
-      </joint>
-      <joint name="${prefix}joint3">
-        <command_interface name="position">
-          <param name="min">-2.7925</param>
-          <param name="max">2.7925</param>
-        </command_interface>
-        <command_interface name="velocity">
-          <param name="min">-4.4435</param>
-          <param name="max">4.4435</param>
-        </command_interface>
-        <command_interface name="effort"/>
-        <state_interface name="position"/>
-        <state_interface name="velocity"/>
-        <state_interface name="effort"/>
-        <!-- initial position for the FakeSystem -->
-        <param name="initial_position">1.57</param>
-        <!-- <param name="initial_position">${initial_positions['joint3']}</param>       -->
-      </joint>
-      <joint name="${prefix}joint4">
-        <command_interface name="position">
-          <param name="min">-2.7925</param>
-          <param name="max">2.7925</param>
-        </command_interface>
-        <command_interface name="velocity">
-          <param name="min">-4.8869</param>
-          <param name="max">4.8869</param>
-        </command_interface>
-        <command_interface name="effort"/>
-        <state_interface name="position"/>
-        <state_interface name="velocity"/>
-        <state_interface name="effort"/>
-        <!-- initial position for the FakeSystem -->
-        <param name="initial_position">0.0</param>
-        <!-- <param name="initial_position">${initial_positions['joint4']}</param>      -->
-      </joint>
-      <joint name="${prefix}joint5">
-        <command_interface name="position">
-          <param name="min">-2.7925</param>
-          <param name="max">2.7925</param>
-        </command_interface>
-        <command_interface name="velocity">
-          <param name="min">-4.8869</param>
-          <param name="max">4.8869</param>
-        </command_interface>
-        <command_interface name="effort"/>
-        <state_interface name="position"/>
-        <state_interface name="velocity"/>
-        <state_interface name="effort"/>
-        <!-- initial position for the FakeSystem -->
-        <param name="initial_position">0.0</param>
-        <!-- <param name="initial_position">${initial_positions['joint5']}</param>         -->
-      </joint>
-      <joint name="${prefix}joint6">
-        <command_interface name="position">
-          <param name="min">-2.7925</param>
-          <param name="max">2.7925</param>
-        </command_interface>
-        <command_interface name="velocity">
-          <param name="min">-4.8869</param>
-          <param name="max">4.8869</param>
-        </command_interface>
-        <command_interface name="effort"/>
-        <state_interface name="position"/>
-        <state_interface name="velocity"/>
-        <state_interface name="effort"/>
-        <!-- initial position for the FakeSystem -->
-        <param name="initial_position">0.0</param>
-        <!-- <param name="initial_position">${initial_positions['joint6']}</param>         -->
-      </joint>
-      <sensor name="${prefix}force_torque_sensor">
-        <state_interface name="force.x"/>
-        <state_interface name="force.y"/>
-        <state_interface name="force.z"/>
-        <state_interface name="torque.x"/>
-        <state_interface name="torque.y"/>
-        <state_interface name="torque.z"/>
-      </sensor>
-<!--       <joint name="${prefix}wrist_force_torque">
-        <command_interface name="tare_force.x"/>
-        <command_interface name="tare_force.y"/>
-        <command_interface name="tare_force.z"/>
-        <command_interface name="tare_torque.x"/>
-        <command_interface name="tare_torque.y"/>
-        <command_interface name="tare_torque.z"/>
-        <xacro:unless value="${use_fake_hardware}">
-          <state_interface name="force.x"/>
-          <state_interface name="force.y"/>
-          <state_interface name="force.z"/>
-          <state_interface name="torque.x"/>
-          <state_interface name="torque.y"/>
-          <state_interface name="torque.z"/>
-          <state_interface name="fts_faults"/>
-          <state_interface name="fts_warnings"/>
-        </xacro:unless>
-      </joint> -->
+      <joint name="joint1">
+        <command_interface name="position">
+          <param name="min">-3.14</param>
+          <param name="max">3.14</param>
+        </command_interface>
+        <command_interface name="velocity">
+          <param name="min">-3.14</param>
+          <param name="max">3.14</param>
+        </command_interface>
+        <command_interface name="acceleration">
+          <param name="min">-3.14</param>
+          <param name="max">3.14</param>
+        </command_interface>
+        <command_interface name="effort">
+          <param name="min">-200.0</param>
+          <param name="max">200.0</param>
+        </command_interface>
+        <state_interface name="position"/>
+        <state_interface name="velocity"/>
+        <state_interface name="acceleration"/>
+        <state_interface name="effort"/>
+        <param name="initial_position">0.0</param>
+      </joint>
+      <joint name="joint2">
+        <command_interface name="position">
+          <param name="min">-3.14</param>
+          <param name="max">3.14</param>
+        </command_interface>
+        <command_interface name="velocity">
+          <param name="min">-3.14</param>
+          <param name="max">3.14</param>
+        </command_interface>
+        <command_interface name="acceleration">
+          <param name="min">-3.14</param>
+          <param name="max">3.14</param>
+        </command_interface>
+        <command_interface name="effort">
+          <param name="min">-200.0</param>
+          <param name="max">200.0</param>
+        </command_interface>
+        <state_interface name="position"/>
+        <state_interface name="velocity"/>
+        <state_interface name="acceleration"/>
+        <state_interface name="effort"/>
+        <param name="initial_position">0.0</param>
+      </joint>
+      <joint name="joint3">
+        <command_interface name="position">
+          <param name="min">-3.14</param>
+          <param name="max">3.14</param>
+        </command_interface>
+        <command_interface name="velocity">
+          <param name="min">-3.14</param>
+          <param name="max">3.14</param>
+        </command_interface>
+        <command_interface name="acceleration">
+          <param name="min">-3.14</param>
+          <param name="max">3.14</param>
+        </command_interface>
+        <command_interface name="effort">
+          <param name="min">-200.0</param>
+          <param name="max">200.0</param>
+        </command_interface>
+        <state_interface name="position"/>
+        <state_interface name="velocity"/>
+        <state_interface name="acceleration"/>
+        <state_interface name="effort"/>
+        <param name="initial_position">1.5</param>
+      </joint>
+      <joint name="joint4">
+        <command_interface name="position">
+          <param name="min">-3.14</param>
+          <param name="max">3.14</param>
+        </command_interface>
+        <command_interface name="velocity">
+          <param name="min">-3.14</param>
+          <param name="max">3.14</param>
+        </command_interface>
+        <command_interface name="acceleration">
+          <param name="min">-3.14</param>
+          <param name="max">3.14</param>
+        </command_interface>
+        <command_interface name="effort">
+          <param name="min">-200.0</param>
+          <param name="max">200.0</param>
+        </command_interface>
+        <state_interface name="position"/>
+        <state_interface name="velocity"/>
+        <state_interface name="acceleration"/>
+        <state_interface name="effort"/>
+        <param name="initial_position">0.0</param>
+      </joint>
+      <joint name="joint5">
+        <command_interface name="position">
+          <param name="min">-3.14</param>
+          <param name="max">3.14</param>
+        </command_interface>
+        <command_interface name="velocity">
+          <param name="min">-3.14</param>
+          <param name="max">3.14</param>
+        </command_interface>
+        <command_interface name="acceleration">
+          <param name="min">-3.14</param>
+          <param name="max">3.14</param>
+        </command_interface>
+        <command_interface name="effort">
+          <param name="min">-200.0</param>
+          <param name="max">200.0</param>
+        </command_interface>
+        <state_interface name="position"/>
+        <state_interface name="velocity"/>
+        <state_interface name="acceleration"/>
+        <state_interface name="effort"/>
+        <param name="initial_position">0.0</param>
+      </joint>
+      <joint name="joint6">
+        <command_interface name="position">
+          <param name="min">-3.14</param>
+          <param name="max">3.14</param>
+        </command_interface>
+        <command_interface name="velocity">
+          <param name="min">-3.14</param>
+          <param name="max">3.14</param>
+        </command_interface>
+        <command_interface name="acceleration">
+          <param name="min">-3.14</param>
+          <param name="max">3.14</param>
+        </command_interface>
+        <command_interface name="effort">
+          <param name="min">-200.0</param>
+          <param name="max">200.0</param>
+        </command_interface>
+        <state_interface name="position"/>
+        <state_interface name="velocity"/>
+        <state_interface name="acceleration"/>
+        <state_interface name="effort"/>
+        <param name="initial_position">0.0</param>
+      </joint>
     </ros2_control>
   </xacro:macro>

File: ur5_description/urdf/ur5.urdf.xacro (robot description, xacro)
@@ -3,23 +3,12 @@
   <!-- Enable setting arguments from the launch file -->
   <xacro:arg name="name" default="ur5"/>
-  <!-- parameters -->
-  <!-- <xacro:arg name="prefix" default="" />
-  <xacro:arg name="robot_ip" default="" />
-  <xacro:arg name="local_ip" default="" />
-  <xacro:arg name="use_fake_hardware" default="false" />
-  <xacro:arg name="fake_sensor_commands" default="false" /> -->
-  <!-- <xacro:arg name="initial_positions_file" default="$(find ur5_description)/config/initial_positions.yaml"/> -->
   <!-- include ur5 macro -->
   <xacro:include filename="$(find ur5_description)/urdf/ur5_joints_links.xacro" />
   <xacro:ur5_joints_links />
+  <!-- include transmissions -->
+  <xacro:include filename="$(find ur5_description)/urdf/ur5_transmissions.xacro" />
+  <xacro:ur5_transmissions />
   <!-- include ur5 ros2_control description -->
-  <!-- <xacro:include filename="$(find ur5_description)/urdf/ur5.ros2_control.xacro" />
-  <xacro:ur5_ros2_control
-    prefix="$(arg prefix)"
-    robot_ip="$(arg robot_ip)"
-    local_ip="$(arg local_ip)"
-    use_fake_hardware="$(arg use_fake_hardware)"
-    fake_sensor_commands="$(arg fake_sensor_commands)"
-    /> -->
-    <!-- initial_positions_file="$(arg initial_positions_file)" -->
+  <xacro:include filename="$(find ur5_description)/urdf/ur5.ros2_control.xacro" />
+  <xacro:ur5_ros2_control />
 </robot>
