Commit message: Remove material definitions from UR5 URDF
Removed material definitions for visual elements in URDF.

File: ur5_description/urdf/ur5_joints_links.xacro (robot description, xacro)
@@ -10,7 +10,4 @@
           <mesh filename="package://ur5_description/meshes/base.dae" />
         </geometry>
-        <material name="LightGrey">
-          <color rgba="0.7 0.7 0.7 1.0" />
-        </material>
       </visual>
       <collision>
@@ -32,7 +29,4 @@
           <mesh filename="package://ur5_description/meshes/shoulder.dae" />
         </geometry>
-        <material name="LightGrey">
-          <color rgba="0.7 0.7 0.7 1.0" />
-        </material>
       </visual>
       <collision>
@@ -55,7 +49,4 @@
           <mesh filename="package://ur5_description/meshes/upperarm.dae" />
         </geometry>
-        <material name="LightGrey">
-          <color rgba="0.7 0.7 0.7 1.0" />
-        </material>
       </visual>
       <collision>
@@ -78,7 +69,4 @@
           <mesh filename="package://ur5_description/meshes/forearm.dae" />
         </geometry>
-        <material name="LightGrey">
-          <color rgba="0.7 0.7 0.7 1.0" />
-        </material>
       </visual>
       <collision>
@@ -101,7 +89,4 @@
           <mesh filename="package://ur5_description/meshes/wrist1.dae" />
         </geometry>
-        <material name="LightGrey">
-          <color rgba="0.7 0.7 0.7 1.0" />
-        </material>
       </visual>
       <collision>
@@ -124,7 +109,4 @@
           <mesh filename="package://ur5_description/meshes/wrist2.dae" />
         </geometry>
-        <material name="LightGrey">
-          <color rgba="0.7 0.7 0.7 1.0" />
-        </material>
       </visual>
       <collision>
@@ -147,7 +129,4 @@
           <mesh filename="package://ur5_description/meshes/wrist3.dae" />
         </geometry>
-        <material name="LightGrey">
-          <color rgba="0.7 0.7 0.7 1.0" />
-        </material>
       </visual>
       <collision>

Commit message: gazebo fortress updated

File: ur5_description/urdf/ur5_joints_links.xacro (robot description, xacro)
@@ -11,10 +11,4 @@
         </geometry>
       </visual>
-      <collision>
-        <origin rpy="0 0 3.141592653589793" xyz="0 0 0" />
-        <geometry>
-          <mesh filename="package://ur5_description/meshes/base.dae" />
-        </geometry>
-      </collision>
       <inertial>
         <mass value="4.0" />
@@ -30,10 +24,4 @@
         </geometry>
       </visual>
-      <collision>
-        <origin rpy="0 0 3.141592653589793" xyz="0 0 0" />
-        <geometry>
-          <mesh filename="package://ur5_description/meshes/shoulder.dae" />
-        </geometry>
-      </collision>
       <inertial>
         <mass value="3.7" />
@@ -50,10 +38,4 @@
         </geometry>
       </visual>
-      <collision>
-        <origin rpy="1.5707963267948966 0 -1.5707963267948966" xyz="0 0 0.138" />
-        <geometry>
-          <mesh filename="package://ur5_description/meshes/upperarm.dae" />
-        </geometry>
-      </collision>
       <inertial>
         <mass value="8.393" />
@@ -70,10 +52,4 @@
         </geometry>
       </visual>
-      <collision>
-        <origin rpy="1.5707963267948966 0 -1.5707963267948966" xyz="0 0 0.007" />
-        <geometry>
-          <mesh filename="package://ur5_description/meshes/forearm.dae" />
-        </geometry>
-      </collision>
       <inertial>
         <mass value="2.275" />
@@ -90,10 +66,4 @@
         </geometry>
       </visual>
-      <collision>
-        <origin rpy="1.5707963267948966 0 0" xyz="0 0 -0.127" />
-        <geometry>
-          <mesh filename="package://ur5_description/meshes/wrist1.dae" />
-        </geometry>
-      </collision>
       <inertial>
         <mass value="1.219" />
@@ -110,10 +80,4 @@
         </geometry>
       </visual>
-      <collision>
-        <origin rpy="0 0 0" xyz="0 0 -0.0997" />
-        <geometry>
-          <mesh filename="package://ur5_description/meshes/wrist2.dae" />
-        </geometry>
-      </collision>
       <inertial>
         <mass value="1.219" />
@@ -130,10 +94,4 @@
         </geometry>
       </visual>
-      <collision>
-        <origin rpy="1.5707963267948966 0 0" xyz="0 0 -0.0989" />
-        <geometry>
-          <mesh filename="package://ur5_description/meshes/wrist3.dae" />
-        </geometry>
-      </collision>
       <inertial>
         <mass value="0.1879" />
@@ -178,5 +136,5 @@
       <origin rpy="0 0 -1.5707" xyz="-0.3922 0 0.1333" />
       <axis xyz="0 0 1" />
-      <limit effort="28.0" lower="-6.283185307179586" upper="6.283185307179586"
+      <limit effort="150.0" lower="-6.283185307179586" upper="6.283185307179586"
         velocity="3.141592653589793" />
     </joint>
@@ -186,5 +144,5 @@
       <origin rpy="1.570796327 0 0" xyz="0 -0.0997 -2.044881182297852e-11" />
       <axis xyz="0 0 1" />
-      <limit effort="28.0" lower="-6.283185307179586" upper="6.283185307179586"
+      <limit effort="150.0" lower="-6.283185307179586" upper="6.283185307179586"
         velocity="3.141592653589793" />
     </joint>
@@ -195,5 +153,5 @@
         xyz="0 0.0996 -2.042830148012698e-11" />
       <axis xyz="0 0 1" />
-      <limit effort="28.0" lower="-6.283185307179586" upper="6.283185307179586"
+      <limit effort="150.0" lower="-6.283185307179586" upper="6.283185307179586"
         velocity="3.141592653589793" />
     </joint>

File: ur5_description/urdf/ur5_ros2_control.xacro (robot description, xacro)
@@ -4,14 +4,17 @@
     <!-- ROS2 Control Plugin-->
     <gazebo>
-      <plugin filename="libgazebo_ros2_control.so" name="gazebo_ros2_control">
-        <robot_param>robot_description</robot_param>
-        <robot_param_node>robot_state_publisher</robot_param_node>
-        <parameters>$(find ur5_description)/config/robot_controllers.yaml</parameters>
+      <plugin filename="gz_ros2_control-system" name="gz_ros2_control::GazeboSimROS2ControlPlugin">
+        <parameters>$(find gazebo_robot_sim)/config/robot_controllers.yaml</parameters>
       </plugin>
     </gazebo>
+    <!-- Initial Positions Config -->
+    <xacro:property
+        name="initial_positions"
+        value="${xacro.load_yaml('$(find ur5_description)/config/initial_positions.yaml')['initial_positions']}"
+    />
     <!-- ROS2 Control Hardware Interface-->
     <ros2_control name="UR5_Arm_Hardware_Interface" type="system">
       <hardware>
-          <plugin>gazebo_ros2_control/GazeboSystem</plugin>
+          <plugin>gz_ros2_control/GazeboSimSystem</plugin>
       </hardware>
       <joint name="joint_1">
@@ -20,16 +23,7 @@
           <param name="max">3.14</param>
         </command_interface>
-        <command_interface name="velocity">
-          <param name="min">-3.14</param>
-          <param name="max">3.14</param>
-        </command_interface>
-        <command_interface name="effort">
-          <param name="min">-200.0</param>
-          <param name="max">200.0</param>
-        </command_interface>
         <state_interface name="position"/>
         <state_interface name="velocity"/>
-        <state_interface name="effort"/>
-        <param name="initial_position">0.0</param>
+        <param name="initial_position">${initial_positions['joint_1']}</param>
       </joint>
       <joint name="joint_2">
@@ -38,16 +32,7 @@
           <param name="max">3.14</param>
         </command_interface>
-        <command_interface name="velocity">
-          <param name="min">-3.14</param>
-          <param name="max">3.14</param>
-        </command_interface>
-        <command_interface name="effort">
-          <param name="min">-200.0</param>
-          <param name="max">200.0</param>
-        </command_interface>
         <state_interface name="position"/>
         <state_interface name="velocity"/>
-        <state_interface name="effort"/>
-        <param name="initial_position">0.0</param>
+        <param name="initial_position">${initial_positions['joint_2']}</param>
       </joint>
       <joint name="joint_3">
@@ -56,16 +41,7 @@
           <param name="max">3.14</param>
         </command_interface>
-        <command_interface name="velocity">
-          <param name="min">-3.14</param>
-          <param name="max">3.14</param>
-        </command_interface>
-        <command_interface name="effort">
-          <param name="min">-200.0</param>
-          <param name="max">200.0</param>
-        </command_interface>
         <state_interface name="position"/>
         <state_interface name="velocity"/>
-        <state_interface name="effort"/>
-        <param name="initial_position">0.0</param>
+        <param name="initial_position">${initial_positions['joint_3']}</param>
       </joint>
       <joint name="joint_4">
@@ -74,16 +50,7 @@
           <param name="max">3.14</param>
         </command_interface>
-        <command_interface name="velocity">
-          <param name="min">-3.14</param>
-          <param name="max">3.14</param>
-        </command_interface>
-        <command_interface name="effort">
-          <param name="min">-200.0</param>
-          <param name="max">200.0</param>
-        </command_interface>
         <state_interface name="position"/>
         <state_interface name="velocity"/>
-        <state_interface name="effort"/>
-        <param name="initial_position">0.0</param>
+        <param name="initial_position">${initial_positions['joint_4']}</param>
       </joint>
       <joint name="joint_5">
@@ -92,16 +59,7 @@
           <param name="max">3.14</param>
         </command_interface>
-        <command_interface name="velocity">
-          <param name="min">-3.14</param>
-          <param name="max">3.14</param>
-        </command_interface>
-        <command_interface name="effort">
-          <param name="min">-200.0</param>
-          <param name="max">200.0</param>
-        </command_interface>
         <state_interface name="position"/>
         <state_interface name="velocity"/>
-        <state_interface name="effort"/>
-        <param name="initial_position">0.0</param>
+        <param name="initial_position">${initial_positions['joint_5']}</param>
       </joint>
       <joint name="joint_6">
@@ -110,16 +68,7 @@
           <param name="max">3.14</param>
         </command_interface>
-        <command_interface name="velocity">
-          <param name="min">-3.14</param>
-          <param name="max">3.14</param>
-        </command_interface>
-        <command_interface name="effort">
-          <param name="min">-200.0</param>
-          <param name="max">200.0</param>
-        </command_interface>
         <state_interface name="position"/>
         <state_interface name="velocity"/>
-        <state_interface name="effort"/>
-        <param name="initial_position">0.0</param>
+        <param name="initial_position">${initial_positions['joint_6']}</param>
       </joint>
     </ros2_control>

Commit message: robot sim developed

File: ur5_description/urdf/ur5_joints_links.xacro (robot description, xacro)
@@ -2,13 +2,23 @@
 <robot xmlns:xacro="http://ros.org/wiki/xacro">
   <xacro:macro name="ur5_joints_links">
-    <!-- links main serial chain -->
     <link name="world" />
+    <joint name="base_fixed_joint" type="fixed">
+      <parent link="world"/>
+      <child link="base_link"/>
+      <origin xyz="0 0 0" rpy="0 0 0"/>
+    </joint>
     <link name="base_link">
       <visual>
         <origin rpy="0 0 3.141592653589793" xyz="0 0 0" />
         <geometry>
-          <mesh filename="package://ur5_description/meshes/base.dae" />
+          <mesh filename="package://ur5_description/meshes/visual/base.dae" />
         </geometry>
       </visual>
+      <collision>
+        <origin rpy="0 0 3.141592653589793" xyz="0 0 0" />
+        <geometry>
+          <mesh filename="package://ur5_description/meshes/collision/base.stl" />
+        </geometry>
+      </collision>
       <inertial>
         <mass value="4.0" />
@@ -17,94 +27,4 @@
       </inertial>
     </link>
-    <link name="shoulder_link">
-      <visual>
-        <origin rpy="0 0 3.141592653589793" xyz="0 0 0" />
-        <geometry>
-          <mesh filename="package://ur5_description/meshes/shoulder.dae" />
-        </geometry>
-      </visual>
-      <inertial>
-        <mass value="3.7" />
-        <origin rpy="0 0 0" xyz="0 0 0" />
-        <inertia ixx="0.010267495893" ixy="0.0" ixz="0.0" iyy="0.010267495893" iyz="0.0"
-          izz="0.00666" />
-      </inertial>
-    </link>
-    <link name="upper_arm_link">
-      <visual>
-        <origin rpy="1.5707963267948966 0 -1.5707963267948966" xyz="0 0 0.138" />
-        <geometry>
-          <mesh filename="package://ur5_description/meshes/upperarm.dae" />
-        </geometry>
-      </visual>
-      <inertial>
-        <mass value="8.393" />
-        <origin rpy="0 1.5707963267948966 0" xyz="-0.2125 0.0 0.138" />
-        <inertia ixx="0.1338857818623325" ixy="0.0" ixz="0.0" iyy="0.1338857818623325" iyz="0.0"
-          izz="0.0151074" />
-      </inertial>
-    </link>
-    <link name="forearm_link">
-      <visual>
-        <origin rpy="1.5707963267948966 0 -1.5707963267948966" xyz="0 0 0.007" />
-        <geometry>
-          <mesh filename="package://ur5_description/meshes/forearm.dae" />
-        </geometry>
-      </visual>
-      <inertial>
-        <mass value="2.275" />
-        <origin rpy="0 1.5707963267948966 0" xyz="-0.1961 0.0 0.007" />
-        <inertia ixx="0.031209355099586295" ixy="0.0" ixz="0.0" iyy="0.031209355099586295" iyz="0.0"
-          izz="0.004095" />
-      </inertial>
-    </link>
-    <link name="wrist_1_link">
-      <visual>
-        <origin rpy="1.5707963267948966 0 0" xyz="0 0 -0.127" />
-        <geometry>
-          <mesh filename="package://ur5_description/meshes/wrist1.dae" />
-        </geometry>
-      </visual>
-      <inertial>
-        <mass value="1.219" />
-        <origin rpy="0 0 0" xyz="0 0 0" />
-        <inertia ixx="0.0025598989760400002" ixy="0.0" ixz="0.0" iyy="0.0025598989760400002"
-          iyz="0.0" izz="0.0021942" />
-      </inertial>
-    </link>
-    <link name="wrist_2_link">
-      <visual>
-        <origin rpy="0 0 0" xyz="0 0 -0.0997" />
-        <geometry>
-          <mesh filename="package://ur5_description/meshes/wrist2.dae" />
-        </geometry>
-      </visual>
-      <inertial>
-        <mass value="1.219" />
-        <origin rpy="0 0 0" xyz="0 0 0" />
-        <inertia ixx="0.0025598989760400002" ixy="0.0" ixz="0.0" iyy="0.0025598989760400002"
-          iyz="0.0" izz="0.0021942" />
-      </inertial>
-    </link>
-    <link name="wrist_3_link">
-      <visual>
-        <origin rpy="1.5707963267948966 0 0" xyz="0 0 -0.0989" />
-        <geometry>
-          <mesh filename="package://ur5_description/meshes/wrist3.dae" />
-        </geometry>
-      </visual>
-      <inertial>
-        <mass value="0.1879" />
-        <origin rpy="0 0 0" xyz="0.0 0.0 -0.0229" />
-        <inertia ixx="9.890410052167731e-05" ixy="0.0" ixz="0.0" iyy="9.890410052167731e-05"
-          iyz="0.0" izz="0.0001321171875" />
-      </inertial>
-    </link>
-    <!-- joints main serial chain -->
-    <joint name="base_fixed_joint" type="fixed">
-      <parent link="world"/>
-      <child link="base_link"/>
-      <origin xyz="0 0 0" rpy="0 0 0"/>
-    </joint>
     <joint name="joint_1" type="revolute">
       <parent link="base_link" />
@@ -112,7 +32,25 @@
       <origin rpy="0 0 0" xyz="0 0 0.1625" />
       <axis xyz="0 0 1" />
-      <limit effort="150.0" lower="-6.283185307179586" upper="6.283185307179586"
-        velocity="3.141592653589793" />
+      <limit effort="150.0" lower="-6.283185307179586" upper="6.283185307179586" velocity="3.141592653589793" />
     </joint>
+    <link name="shoulder_link">
+      <visual>
+        <origin rpy="0 0 3.141592653589793" xyz="0 0 0" />
+        <geometry>
+          <mesh filename="package://ur5_description/meshes/visual/shoulder.dae" />
+        </geometry>
+      </visual>
+      <collision>
+        <origin rpy="0 0 3.141592653589793" xyz="0 0 0" />
+        <geometry>
+          <mesh filename="package://ur5_description/meshes/collision/shoulder.stl" />
+        </geometry>
+      </collision>
+      <inertial>
+        <mass value="3.7" />
+        <origin rpy="0 0 0" xyz="0 0 0" />
+        <inertia ixx="0.010267495893" ixy="0.0" ixz="0.0" iyy="0.010267495893" iyz="0.0" izz="0.00666" />
+      </inertial>
+    </link>
     <joint name="joint_2" type="revolute">
       <parent link="shoulder_link" />
@@ -120,7 +58,25 @@
       <origin rpy="1.5707 1.5707 0" xyz="0 0 0" />
       <axis xyz="0 0 1" />
-      <limit effort="150.0" lower="-6.283185307179586" upper="6.283185307179586"
-        velocity="3.141592653589793" />
+      <limit effort="150.0" lower="-6.283185307179586" upper="6.283185307179586" velocity="3.141592653589793" />
     </joint>
+    <link name="upper_arm_link">
+      <visual>
+        <origin rpy="1.5707963267948966 0 -1.5707963267948966" xyz="0 0 0.138" />
+        <geometry>
+          <mesh filename="package://ur5_description/meshes/visual/upperarm.dae" />
+        </geometry>
+      </visual>
+      <collision>
+        <origin rpy="1.5707963267948966 0 -1.5707963267948966" xyz="0 0 0.138" />
+        <geometry>
+          <mesh filename="package://ur5_description/meshes/collision/upperarm.stl" />
+        </geometry>
+      </collision>
+      <inertial>
+        <mass value="8.393" />
+        <origin rpy="0 1.5707963267948966 0" xyz="-0.2125 0.0 0.138" />
+        <inertia ixx="0.1338857818623325" ixy="0.0" ixz="0.0" iyy="0.1338857818623325" iyz="0.0" izz="0.0151074" />
+      </inertial>
+    </link>
     <joint name="joint_3" type="revolute">
       <parent link="upper_arm_link" />
@@ -128,7 +84,25 @@
       <origin rpy="0 0 0" xyz="-0.425 0 0" />
       <axis xyz="0 0 1" />
-      <limit effort="150.0" lower="-3.141592653589793" upper="3.141592653589793"
-        velocity="3.141592653589793" />
+      <limit effort="150.0" lower="-3.141592653589793" upper="3.141592653589793" velocity="3.141592653589793" />
     </joint>
+    <link name="forearm_link">
+      <visual>
+        <origin rpy="1.5707963267948966 0 -1.5707963267948966" xyz="0 0 0.007" />
+        <geometry>
+          <mesh filename="package://ur5_description/meshes/visual/forearm.dae" />
+        </geometry>
+      </visual>
+      <collision>
+        <origin rpy="1.5707963267948966 0 -1.5707963267948966" xyz="0 0 0.007" />
+        <geometry>
+          <mesh filename="package://ur5_description/meshes/collision/forearm.stl" />
+        </geometry>
+      </collision>
+      <inertial>
+        <mass value="2.275" />
+        <origin rpy="0 1.5707963267948966 0" xyz="-0.1961 0.0 0.007" />
+        <inertia ixx="0.031209355099586295" ixy="0.0" ixz="0.0" iyy="0.031209355099586295" iyz="0.0" izz="0.004095" />
+      </inertial>
+    </link>
     <joint name="joint_4" type="revolute">
       <parent link="forearm_link" />
@@ -136,7 +110,25 @@
       <origin rpy="0 0 -1.5707" xyz="-0.3922 0 0.1333" />
       <axis xyz="0 0 1" />
-      <limit effort="150.0" lower="-6.283185307179586" upper="6.283185307179586"
-        velocity="3.141592653589793" />
+      <limit effort="150.0" lower="-6.283185307179586" upper="6.283185307179586" velocity="3.141592653589793" />
     </joint>
+    <link name="wrist_1_link">
+      <visual>
+        <origin rpy="1.5707963267948966 0 0" xyz="0 0 -0.127" />
+        <geometry>
+          <mesh filename="package://ur5_description/meshes/visual/wrist1.dae" />
+        </geometry>
+      </visual>
+      <collision>
+        <origin rpy="1.5707963267948966 0 0" xyz="0 0 -0.127" />
+        <geometry>
+          <mesh filename="package://ur5_description/meshes/collision/wrist1.stl" />
+        </geometry>
+      </collision>
+      <inertial>
+        <mass value="1.219" />
+        <origin rpy="0 0 0" xyz="0 0 0" />
+        <inertia ixx="0.0025598989760400002" ixy="0.0" ixz="0.0" iyy="0.0025598989760400002" iyz="0.0" izz="0.0021942" />
+      </inertial>
+    </link>
     <joint name="joint_5" type="revolute">
       <parent link="wrist_1_link" />
@@ -144,16 +136,51 @@
       <origin rpy="1.570796327 0 0" xyz="0 -0.0997 -2.044881182297852e-11" />
       <axis xyz="0 0 1" />
-      <limit effort="150.0" lower="-6.283185307179586" upper="6.283185307179586"
-        velocity="3.141592653589793" />
+      <limit effort="150.0" lower="-6.283185307179586" upper="6.283185307179586" velocity="3.141592653589793" />
     </joint>
+    <link name="wrist_2_link">
+      <visual>
+        <origin rpy="0 0 0" xyz="0 0 -0.0997" />
+        <geometry>
+          <mesh filename="package://ur5_description/meshes/visual/wrist2.dae" />
+        </geometry>
+      </visual>
+      <collision>
+        <origin rpy="0 0 0" xyz="0 0 -0.0997" />
+        <geometry>
+          <mesh filename="package://ur5_description/meshes/collision/wrist2.stl" />
+        </geometry>
+      </collision>
+      <inertial>
+        <mass value="1.219" />
+        <origin rpy="0 0 0" xyz="0 0 0" />
+        <inertia ixx="0.0025598989760400002" ixy="0.0" ixz="0.0" iyy="0.0025598989760400002" iyz="0.0" izz="0.0021942" />
+      </inertial>
+    </link>
     <joint name="joint_6" type="revolute">
       <parent link="wrist_2_link" />
       <child link="wrist_3_link" />
-      <origin rpy="1.570796326589793 3.141592653589793 3.141592653589793"
-        xyz="0 0.0996 -2.042830148012698e-11" />
+      <origin rpy="1.570796326589793 3.141592653589793 3.141592653589793" xyz="0 0.0996 -2.042830148012698e-11" />
       <axis xyz="0 0 1" />
-      <limit effort="150.0" lower="-6.283185307179586" upper="6.283185307179586"
-        velocity="3.141592653589793" />
+      <limit effort="150.0" lower="-6.283185307179586" upper="6.283185307179586" velocity="3.141592653589793" />
     </joint>
+    <link name="wrist_3_link">
+      <visual>
+        <origin rpy="1.5707963267948966 0 0" xyz="0 0 -0.0989" />
+        <geometry>
+          <mesh filename="package://ur5_description/meshes/visual/wrist3.dae" />
+        </geometry>
+      </visual>
+      <collision>
+        <origin rpy="1.5707963267948966 0 0" xyz="0 0 -0.0989" />
+        <geometry>
+          <mesh filename="package://ur5_description/meshes/collision/wrist3.stl" />
+        </geometry>
+      </collision>
+      <inertial>
+        <mass value="0.1879" />
+        <origin rpy="0 0 0" xyz="0.0 0.0 -0.0229" />
+        <inertia ixx="9.890410052167731e-05" ixy="0.0" ixz="0.0" iyy="9.890410052167731e-05" iyz="0.0" izz="0.0001321171875" />
+      </inertial>
+    </link>
   </xacro:macro>
 </robot>

File: ur5_description/urdf/ur5_urdf.xacro (robot description, xacro)
@@ -1,4 +1,6 @@
 <?xml version="1.0" ?>
 <robot xmlns:xacro="http://ros.org/wiki/xacro" name="ur5">
+  <!-- Enable setting arguments from the launch file -->
+  <!-- <xacro:arg name="name" default="ur5"/> -->
   <!-- include ur5 macro -->
   <xacro:include filename="$(find ur5_description)/urdf/ur5_joints_links.xacro" />
